Commit message: Multiple sensors added

File: description/robot.urdf.xacro (robot description, xacro)
@@ -1,7 +1,13 @@
 <?xml version="1.0"?>
-<robot xmlns:xacro="http://www.ros.org/wiki/xacro"  name="robot">
+<robot xmlns:xacro="http://www.ros.org/wiki/xacro" name="robot">
     <!-- Example link -->
+    <xacro:include filename="inertial_macros.xacro"/>
+    <xacro:include filename="properties.xacro"/>
     <xacro:include filename="robot_core.xacro"/>
-        <!-- Example link -->
-    <link name="base_link"></link>
+    <xacro:include filename="gazebo_control.xacro"/>
+    <xacro:include filename="imu.xacro"/>
+    <xacro:include filename="lidar.xacro"/>
+    <!--xacro:include filename="camera.xacro"/-->
+    <xacro:include filename="kinect.xacro"/>
+    <!-- Example link -->
 </robot>
