Commit message: ackerman car with ros2 controll added

File: description/robot_core.xacro (robot description, xacro)
@@ -54,5 +54,5 @@
     <!-- right wheel joint -->
     <joint name="right_wheel_joint" type="continuous">
-        <parent link="base_link"/>
+        <parent link="chassis_link"/>
         <child link="right_wheel"/>
         <origin xyz="0 -0.175 0" rpy="${pi/2} 0 0"/>

File: description_ackerman/kinect.xacro (robot description, xacro)
@@ -4,6 +4,6 @@
     <joint name="kinect_joint" type="fixed">
         <axis xyz="0 0 0" />
-        <origin xyz="${0.3+kinect_link/4} 0 ${0.15-kinect_link/2}" rpy="0 0 0"/>
-        <parent link="chassis"/>
+        <origin xyz="${0.3+kinect_link/4} 0 ${0.05+kinect_link/2}" rpy="0 0 0"/>
+        <parent link="chassis_link"/>
         <child link="kinect_link"/>
     </joint>

File: description_ackerman/lidar.xacro (robot description, xacro)
@@ -3,7 +3,7 @@
     <!-- lidar joint -->
     <joint name="laser_joint" type="fixed">
-        <parent link="chassis"/>
+        <parent link="chassis_link"/>
         <child link="laser_frame"/>
-        <origin xyz="0.1 0 0.17" rpy="0 0 0"/>
+        <origin xyz="-0.25 0 0.125" rpy="0 0 0"/>
     </joint>
     <!-- laser_frame -->
