Commit message: bycicle steering

File: description_ackerman/ackerman_robot_core.urdf.xacro (robot description, xacro)
@@ -2,6 +2,4 @@
 <robot name="ackrm_robot"
   xmlns:xacro="http://ros.org/wiki/xacro">
-  <!--MATERIALS-->
-  <!-- XACRO PROPERTIES -->
   <xacro:property name="PI" value="3.1415926535897931"/>
   <xacro:property name="chassis_length" value="0.8" />
@@ -12,7 +10,5 @@
   <xacro:property name="wheel_heigth" value="0.05" />
   <xacro:property name="wheel_mass" value="${pi*wheel_radius*wheel_radius*wheel_heigth*500}" />
-  <!-- XACRO LIBRARIES -->
   <xacro:include filename="wheel_macros.xacro" />
-<!-- Example link -->
 <link name="base_link">
 </link>
@@ -22,5 +18,4 @@
   <origin xyz="0 0 0"/>
 </joint>
-  <!-- chassis LINK DEFINITION -->
   <link name="chassis_link">
     <visual>
@@ -39,14 +34,21 @@
     </xacro:inertial_box>
   </link>
-  <!-- VIRTUAL WHEELS-->
-  <!-- virtual front wheel -->
   <link name="virtual_front_wheel">
     <visual>
       <origin xyz="0 0 0" rpy="${PI/2} 0 ${PI/2}"/>
       <geometry>
-        <cylinder length="0.01" radius="${wheel_radius}"/>
+        <cylinder length="0.4" radius="${wheel_radius}"/>
       </geometry>
       <material name="invisible"/>
     </visual>
+    <xacro:inertial_cylinder mass="0.1" length="0.4" radius="0.1">
+      <origin xyz="0 0 0" rpy="${PI/2} 0 ${PI/2}"/>
+    </xacro:inertial_cylinder>
+    <collision>
+      <origin xyz="0 0 0" rpy="${PI/2} 0 ${PI/2}" />
+      <geometry>
+          <cylinder radius="0.1" length="0.4"/>
+      </geometry>
+    </collision>
   </link>
   <joint name="virtual_front_wheel_joint" type="revolute">
@@ -58,13 +60,21 @@
     <dynamics damping="0.2"/>
   </joint>
-  <!-- virtual back wheel -->
   <link name="virtual_rear_wheel">
     <visual>
       <origin xyz="0 0 0" rpy="${PI/2} 0 ${PI/2}"/>
       <geometry>
-        <cylinder length="0.01" radius="${wheel_radius}"/>
+        <cylinder length="0.4" radius="${wheel_radius}"/>
       </geometry>
       <material name="invisible"/>
     </visual>
+    <xacro:inertial_cylinder mass="0.1" length="0.4" radius="0.1">
+      <origin xyz="0 0 0" rpy="${PI/2} 0 ${PI/2}"/>
+    </xacro:inertial_cylinder>
+    <collision>
+      <origin xyz="0 0 0" rpy="${PI/2} 0 ${PI/2}" />
+      <geometry>
+          <cylinder radius="0.1" length="0.4"/>
+      </geometry>
+    </collision>
   </link>
   <joint name="virtual_rear_wheel_joint" type="continuous">
@@ -76,40 +86,3 @@
     <dynamics damping="0.2"/>
   </joint>
-  <!-- WHEELS MACRO CALL -->
-  <xacro:cylinder_wheel name="rear_right"
-    wr="${wheel_radius}"
-    wh="${wheel_heigth}"
-    wm="${wheel_mass}"
-    parent="chassis_link"
-    xpos="-0.35"
-    ypos="-0.35"
-    mimic="rear"
-    axis= "0 1 0"/>
-  <xacro:cylinder_wheel name="rear_left"
-    wr="${wheel_radius}"
-    wh="${wheel_heigth}"
-    wm="${wheel_mass}"
-    parent="chassis_link"
-    xpos="-0.35"
-    ypos="0.35"
-    mimic="rear"
-    axis="0 1 0"/>
-  <xacro:cylinder_wheel name="front_right"
-    wr="${wheel_radius}"
-    wh="${wheel_heigth}"
-    wm="${wheel_mass}"
-    parent="chassis_link"
-    xpos="0.35"
-    ypos="0.35"
-    mimic="front"
-    axis="0 0 1"/>
-  <xacro:cylinder_wheel name="front_left"
-    wr="${wheel_radius}"
-    wh="${wheel_heigth}"
-    wm="${wheel_mass}"
-    parent="chassis_link"
-    xpos="0.35"
-    ypos="-0.35"
-    mimic="front"
-    axis="0 0 1"/>
 </robot>

File: description_ackerman/camera.xacro (robot description, xacro)
@@ -1,5 +1,5 @@
 <?xml version="1.0"?>
 <robot xmlns:xacro="http://www.ros.org/wiki/xacro">
-    <xacro:property name="camera_link" value="0.05" /> <!-- Size of square 'camera' box -->
+    <xacro:property name="camera_link" value="0.05" />
     <joint name="camera_joint" type="fixed">
         <axis xyz="0 1 0" />
@@ -8,5 +8,4 @@
         <child link="camera_link"/>
     </joint>
-    <!-- Camera -->
     <link name="camera_link">
         <visual>
@@ -27,5 +26,4 @@
         </xacro:inertial_box>
     </link>
-    <!-- camera -->
   <gazebo reference="camera_link">
     <material>Gazebo/Blue</material>
@@ -46,7 +44,4 @@
         <noise>
           <type>gaussian</type>
-          <!-- Noise is sampled independently per pixel on each frame.
-               That pixel's noise value is added to each of its color
-               channels, which at that point lie in the range [0,1]. -->
           <mean>0.0</mean>
           <stddev>0.007</stddev>

File: description_ackerman/imu.xacro (robot description, xacro)
@@ -1,5 +1,4 @@
 <?xml version="1.0"?>
 <robot xmlns:xacro="http://www.ros.org/wiki/xacro">
-    <!-- Imu_frame -->
     <link name="imu_frame">
         <visual>
@@ -20,5 +19,4 @@
         </collision>
     </link>
-    <!-- Imu joint -->
     <joint name="imu_joint" type="fixed">
         <parent link="chassis_link"/>
@@ -33,21 +31,15 @@
             <update_rate>20</update_rate>
             <visualize>true</visualize>
-            <!--Sensor will be published for the default topic-->
             <topic>__default_topic__</topic>
             <plugin filename="libgazebo_ros_imu_sensor.so" name="imu_plugin">
-                <!--Sensor data will be published for the default topic-->
                 <topicName>imu</topicName>
                 <bodyName>imu_frame</bodyName>
                 <updateRateHZ>20.0</updateRateHZ>
                 <gaussianNoise>0.0</gaussianNoise>
-                <!--Offsets from the reference link reference frame-->
                 <xyzOffset>0 0 0</xyzOffset>
                 <rpyOffset>0 0 0</rpyOffset>
                 <frameName>imu_frame</frameName>
-                <!--Sensor doesn't calibrate to the initial position-->
-                <!--So world is tajen as reference-->
                 <initialOrientationAsReference>false</initialOrientationAsReference>
                 <ros>
-                    <!--Output topic: scan-->
                     <remapping>~/out:=/imu</remapping>
                 </ros>

File: description_ackerman/inertial_macros.xacro (robot description, xacro)
@@ -1,6 +1,4 @@
 <?xml version="1.0"?>
 <robot xmlns:xacro="http://www.ros.org/wiki/xacro" >
-    <!-- Specify some standard inertial calculations https://en.wikipedia.org/wiki/List_of_moments_of_inertia -->
-    <!-- These make use of xacro's mathematical functionality -->
     <xacro:macro name="inertial_sphere" params="mass radius *origin">
         <inertial>

File: description_ackerman/kinect.xacro (robot description, xacro)
@@ -1,5 +1,5 @@
 <?xml version="1.0"?>
 <robot xmlns:xacro="http://www.ros.org/wiki/xacro">
-    <xacro:property name="kinect_link" value="0.05" /> <!-- Size of square 'kinect' box -->
+    <xacro:property name="kinect_link" value="0.05" />
     <joint name="kinect_joint" type="fixed">
         <axis xyz="0 0 0" />
@@ -8,5 +8,4 @@
         <child link="kinect_link"/>
     </joint>
-    <!-- kinect -->
     <link name="kinect_link">
         <visual>
@@ -31,6 +30,5 @@
         <parent link="kinect_link"/>
         <child link="kinect_optical_link"/>
-        <!-- Optical frame: X forward, Y left, Z down -->
-        <origin xyz="0 0 0" rpy="-1.5708 0 -1.5708"/> <!-- -90° around X, then -90° around Z -->
+        <origin xyz="0 0 0" rpy="-1.5708 0 -1.5708"/>
     </joint>
     <gazebo reference="kinect_link">

File: description_ackerman/lidar.xacro (robot description, xacro)
@@ -1,5 +1,4 @@
 <?xml version="1.0"?>
 <robot xmlns:xacro="http://www.ros.org/wiki/xacro">
-    <!-- lidar joint -->
     <joint name="laser_joint" type="fixed">
         <parent link="chassis_link"/>
@@ -7,5 +6,4 @@
         <origin xyz="-0.25 0 0.125" rpy="0 0 0"/>
     </joint>
-    <!-- laser_frame -->
     <link name="laser_frame">
         <visual>
@@ -33,7 +31,5 @@
                 <scan>
                     <horizontal>
-                        <!--samples> is the number of simulated lidar rays to generate per complete laser sweep cycle.-->
                         <samples>360</samples>
-                        <!--resolution>: this number is multiplied by samples to determine the number range data points.-->
                         <resolution>1</resolution>
                         <min_angle>-3.14</min_angle>

File: description_ackerman/properties.xacro (robot description, xacro)
@@ -1,5 +1,4 @@
 <?xml version="1.0"?>
 <robot xmlns:xacro="http://www.ros.org/wiki/xacro">
-    <!-- Color Definitions -->
     <material name="white">
         <color rgba= "1 1 1 1"/>

File: description_ackerman/ros_control.xacro (robot description, xacro)
@@ -3,10 +3,11 @@
     <ros2_control name="steering_control" type="system">
       <hardware>
-        <plugin>ros2_control_demo_example_11/CarlikeBotSystemHardware</plugin>
-        <param name="example_param_hw_start_duration_sec">0</param>
-        <param name="example_param_hw_stop_duration_sec">3.0</param>
+        <plugin>gazebo_ros2_control/GazeboSystem</plugin>
       </hardware>
       <joint name="virtual_front_wheel_joint">
-        <command_interface name="position"/>
+        <command_interface name="position">
+          <param name="min">-0.785</param>
+          <param name="max">0.785</param>
+        </command_interface>
         <state_interface name="position"/>
       </joint>
@@ -20,4 +21,8 @@
       <plugin  name="gazebo_ros2_control" filename="libgazebo_ros2_control.so">
         <parameters>$(find amr_sim_2511_golf)/config/controller.yaml</parameters>
+        <ros>
+          <remapping> /bicycle_steering_controller/tf_odometry:=/tf </remapping>
+          <remapping> /bicycle_steering_controller/reference:=/cmd_vel_stamped </remapping>
+        </ros>
       </plugin>
     </gazebo>

Commit message: bycicle steering "real size"

File: description_ackerman/ackerman_robot_core.urdf.xacro (robot description, xacro)
@@ -3,11 +3,14 @@
   xmlns:xacro="http://ros.org/wiki/xacro">
   <xacro:property name="PI" value="3.1415926535897931"/>
-  <xacro:property name="chassis_length" value="0.8" />
-  <xacro:property name="chassis_width" value="0.4" />
-  <xacro:property name="chassis_heigth" value="0.1" />
-  <xacro:property name="chassis_mass" value="${chassis_length*chassis_width*chassis_heigth*500}" />
-  <xacro:property name="wheel_radius" value="0.1" />
-  <xacro:property name="wheel_heigth" value="0.05" />
-  <xacro:property name="wheel_mass" value="${pi*wheel_radius*wheel_radius*wheel_heigth*500}" />
+  <xacro:property name="chassis_length" value="0.22" />
+  <xacro:property name="chassis_width" value="0.14" />
+  <xacro:property name="chassis_heigth" value="0.03" />
+  <xacro:property name="chassis_mass" value="${chassis_length*chassis_width*chassis_heigth*5000}" />
+  <xacro:property name="wheel_radius" value="0.035" />
+  <xacro:property name="wheel_length" value="0.03" />
+  <xacro:property name="wheel_mass" value="${pi*wheel_radius*wheel_radius*wheel_length*500}" />
+  <xacro:property name="virtual_wheel_radius" value="0.005" />
+  <xacro:property name="virtual_wheel_length" value="0.001" />
+  <xacro:property name="virtual_wheel_mass" value="0.001" />
   <xacro:include filename="wheel_macros.xacro" />
 <link name="base_link">
@@ -34,13 +37,13 @@
     </xacro:inertial_box>
   </link>
-  <link name="virtual_front_wheel">
+  <link name="front_wheel_steering">
     <visual>
       <origin xyz="0 0 0" rpy="${PI/2} 0 ${PI/2}"/>
       <geometry>
-        <cylinder length="0.4" radius="${wheel_radius}"/>
+        <cylinder length="${wheel_length}" radius="${wheel_radius-0.01}"/>
       </geometry>
       <material name="invisible"/>
     </visual>
-    <xacro:inertial_cylinder mass="0.1" length="0.4" radius="0.1">
+    <xacro:inertial_cylinder mass="${wheel_mass}" length="${wheel_length}" radius="${wheel_radius-0.01}">
       <origin xyz="0 0 0" rpy="${PI/2} 0 ${PI/2}"/>
     </xacro:inertial_cylinder>
@@ -48,25 +51,24 @@
       <origin xyz="0 0 0" rpy="${PI/2} 0 ${PI/2}" />
       <geometry>
-          <cylinder radius="0.1" length="0.4"/>
+          <cylinder radius="${wheel_radius-0.01}" length="${wheel_length}"/>
       </geometry>
     </collision>
   </link>
-  <joint name="virtual_front_wheel_joint" type="revolute">
+  <joint name="front_wheel_steering_joint" type="revolute">
     <parent link="chassis_link"/>
-    <child link="virtual_front_wheel"/>
-    <origin xyz="0.35 0 0" rpy="0 0 ${PI/2}"/>
+    <child link="front_wheel_steering"/>
+    <origin xyz="${chassis_length/2+wheel_radius+0.01} 0 0" rpy="0 0 ${PI/2}"/>
     <axis xyz="0 0 1"/>
     <limit lower="-${PI/4}" upper="${PI/4}" effort="100.0" velocity="0.0"/>
-    <dynamics damping="0.2"/>
+    <dynamics damping="0.03"/>
   </joint>
-  <link name="virtual_rear_wheel">
+  <link name="front_wheel">
     <visual>
       <origin xyz="0 0 0" rpy="${PI/2} 0 ${PI/2}"/>
       <geometry>
-        <cylinder length="0.4" radius="${wheel_radius}"/>
+        <cylinder length="${wheel_length}" radius="${wheel_radius}"/>
       </geometry>
-      <material name="invisible"/>
     </visual>
-    <xacro:inertial_cylinder mass="0.1" length="0.4" radius="0.1">
+    <xacro:inertial_cylinder mass="${wheel_mass}" length="${wheel_length}" radius="${wheel_radius}">
       <origin xyz="0 0 0" rpy="${PI/2} 0 ${PI/2}"/>
     </xacro:inertial_cylinder>
@@ -74,5 +76,29 @@
       <origin xyz="0 0 0" rpy="${PI/2} 0 ${PI/2}" />
       <geometry>
-          <cylinder radius="0.1" length="0.4"/>
+          <cylinder radius="${wheel_radius}" length="${wheel_length}"/>
+      </geometry>
+    </collision>
+  </link>
+  <joint name="front_wheel_joint" type="continuous">
+    <parent link="front_wheel_steering"/>
+    <child link="front_wheel"/>
+    <origin xyz="0 0 0" rpy="0 0 0"/>
+    <axis xyz="1 0 0"/>
+  </joint>"
+  <link name="virtual_rear_wheel">
+    <visual>
+      <origin xyz="0 0 0" rpy="${PI/2} 0 ${PI/2}"/>
+      <geometry>
+        <cylinder length="${virtual_wheel_length}" radius="${virtual_wheel_radius}"/>
+      </geometry>
+      <material name="invisible"/>
+    </visual>
+    <xacro:inertial_cylinder mass="${virtual_wheel_mass}" length="${virtual_wheel_length}" radius="${virtual_wheel_radius}">
+      <origin xyz="0 0 0" rpy="${PI/2} 0 ${PI/2}"/>
+    </xacro:inertial_cylinder>
+    <collision>
+      <origin xyz="0 0 0" rpy="${PI/2} 0 ${PI/2}" />
+      <geometry>
+          <cylinder radius="${virtual_wheel_radius}" length="${virtual_wheel_length}"/>
       </geometry>
     </collision>
@@ -81,8 +107,54 @@
     <parent link="chassis_link"/>
     <child link="virtual_rear_wheel"/>
-    <origin xyz="-0.35 0 0" rpy="0 0 ${PI/2}"/>
+    <origin xyz="-${chassis_length/2-wheel_radius} 0 0" rpy="0 0 ${PI/2}"/>
     <axis xyz="1 0 0"/>
     <limit effort="100.0" velocity="100.0"/>
-    <dynamics damping="0.2"/>
+    <dynamics damping="0.03"/>
+  </joint>
+  <link name="right_rear_wheel">
+    <visual>
+      <origin xyz="0 0 0" rpy="${PI/2} 0 ${PI/2}"/>
+      <geometry>
+        <cylinder length="${wheel_length}" radius="${wheel_radius}"/>
+      </geometry>
+    </visual>
+    <xacro:inertial_cylinder mass="${wheel_mass}" length="${wheel_length}" radius="${wheel_radius}">
+      <origin xyz="0 0 0" rpy="${PI/2} 0 ${PI/2}"/>
+    </xacro:inertial_cylinder>
+    <collision>
+      <origin xyz="0 0 0" rpy="${PI/2} 0 ${PI/2}" />
+      <geometry>
+          <cylinder radius="${wheel_radius}" length="${wheel_length}"/>
+      </geometry>
+    </collision>
+  </link>
+  <joint name="right_rear_wheel_joint" type="fixed">
+    <parent link="virtual_rear_wheel"/>
+    <child link="right_rear_wheel"/>
+    <origin xyz="${chassis_width/2+wheel_length/2+0.01} 0 0" rpy="0 0 0"/>
+    <axis xyz="1 0 0"/>
+  </joint>
+  <link name="left_rear_wheel">
+    <visual>
+      <origin xyz="0 0 0" rpy="${PI/2} 0 ${PI/2}"/>
+      <geometry>
+        <cylinder length="${wheel_length}" radius="${wheel_radius}"/>
+      </geometry>
+    </visual>
+    <xacro:inertial_cylinder mass="${wheel_mass}" length="${wheel_length}" radius="${wheel_radius}">
+      <origin xyz="0 0 0" rpy="${PI/2} 0 ${PI/2}"/>
+    </xacro:inertial_cylinder>
+    <collision>
+      <origin xyz="0 0 0" rpy="${PI/2} 0 ${PI/2}" />
+      <geometry>
+          <cylinder radius="${wheel_radius}" length="${wheel_length}"/>
+      </geometry>
+    </collision>
+  </link>
+  <joint name="left_rear_wheel_joint" type="fixed">
+    <parent link="virtual_rear_wheel"/>
+    <child link="left_rear_wheel"/>
+    <origin xyz="-${chassis_width/2+wheel_length/2+0.01} 0 0" rpy="0 0 0"/>
+    <axis xyz="1 0 0"/>
   </joint>
 </robot>

File: description_ackerman/imu.xacro (robot description, xacro)
@@ -1,13 +1,17 @@
 <?xml version="1.0"?>
 <robot xmlns:xacro="http://www.ros.org/wiki/xacro">
+    <xacro:property name="imu_length" value="0.01" />
+    <xacro:property name="imu_heigth" value="0.005" />
+    <xacro:property name="imu_width" value="0.01" />
+    <xacro:property name="imu_mass" value="0.001" />
     <link name="imu_frame">
         <visual>
             <origin xyz="0 0 0"/>
             <geometry>
-                <box size="0.01 0.01 0.005"/>
+                <box size="${imu_width} ${imu_length} ${imu_heigth}"/>
             </geometry>
             <material name="red"/>
         </visual>
-        <xacro:inertial_box mass="0.005" x="0.01" y="0.01" z="0.005">
+        <xacro:inertial_box mass="${imu_mass}" x="${imu_width}" y="${imu_length}" z="${imu_heigth}">
             <origin xyz="0 0 0" rpy="0 0 0"/>
         </xacro:inertial_box>
@@ -15,5 +19,5 @@
             <origin xyz="0 0 0"/>
             <geometry>
-                <box size="0.1 0.1 0.01"/>
+                <box size="${imu_width} ${imu_length} ${imu_heigth}"/>
             </geometry>
         </collision>
@@ -22,5 +26,5 @@
         <parent link="chassis_link"/>
         <child link="imu_frame"/>
-        <origin xyz="0 0 0.052" rpy="0 0 0"/>
+        <origin xyz="0 0 ${chassis_heigth/2+imu_heigth/2}" rpy="0 0 0"/>
     </joint>
     <gazebo reference="imu_frame">

File: description_ackerman/kinect.xacro (robot description, xacro)
@@ -1,8 +1,11 @@
 <?xml version="1.0"?>
 <robot xmlns:xacro="http://www.ros.org/wiki/xacro">
-    <xacro:property name="kinect_link" value="0.05" />
+    <xacro:property name="kinect_length" value="0.09" />
+    <xacro:property name="kinect_heigth" value="0.03" />
+    <xacro:property name="kinect_width" value="0.03" />
+    <xacro:property name="kinect_mass" value="0.5" />
     <joint name="kinect_joint" type="fixed">
         <axis xyz="0 0 0" />
-        <origin xyz="${0.3+kinect_link/4} 0 ${0.05+kinect_link/2}" rpy="0 0 0"/>
+        <origin xyz="${chassis_length/2-kinect_width/2} 0 ${wheel_radius+kinect_heigth/2}" rpy="0 0 0"/>
         <parent link="chassis_link"/>
         <child link="kinect_link"/>
@@ -12,5 +15,5 @@
             <origin xyz="0 0 0" rpy="0 0 0"/>
             <geometry>
-        <box size="${kinect_link/2} ${kinect_link*3} ${kinect_link}"/>
+        <box size="${kinect_width} ${kinect_length} ${kinect_heigth}"/>
             </geometry>
             <material name="blue"/>
@@ -19,8 +22,8 @@
             <origin xyz="0 0 0" rpy="0 0 0"/>
             <geometry>
-        <box size="${kinect_link/2} ${kinect_link*3} ${kinect_link}"/>
+        <box size="${kinect_width} ${kinect_length} ${kinect_heigth}"/>
             </geometry>
         </collision>
-        <xacro:inertial_box mass="0.005" x="${kinect_link/2}" y="${kinect_link*3}" z="${kinect_link}">
+        <xacro:inertial_box mass="${kinect_mass}" x="${kinect_width}" y="${kinect_length}" z="${kinect_heigth}">
             <origin xyz="0 0 0" rpy="0 0 0"/>
         </xacro:inertial_box>
@@ -30,5 +33,5 @@
         <parent link="kinect_link"/>
         <child link="kinect_optical_link"/>
-        <origin xyz="0 0 0" rpy="-1.5708 0 -1.5708"/>
+        <origin xyz="0 0 0" rpy="-${PI/2} 0 -${PI/2}"/>
     </joint>
     <gazebo reference="kinect_link">

File: description_ackerman/lidar.xacro (robot description, xacro)
@@ -1,13 +1,16 @@
 <?xml version="1.0"?>
 <robot xmlns:xacro="http://www.ros.org/wiki/xacro">
+    <xacro:property name="lidar_radius" value="0.035" />
+    <xacro:property name="lidar_length" value="0.03" />
+    <xacro:property name="lidar_mass" value="0.1" />
     <joint name="laser_joint" type="fixed">
         <parent link="chassis_link"/>
         <child link="laser_frame"/>
-        <origin xyz="-0.25 0 0.125" rpy="0 0 0"/>
+        <origin xyz="0 0 ${wheel_radius*3-lidar_length/2}" rpy="0 0 0"/>
     </joint>
     <link name="laser_frame">
         <visual>
             <geometry>
-                <cylinder radius="0.05" length="0.04"/>
+                <cylinder radius="${lidar_radius}" length="${lidar_length}"/>
             </geometry>
             <material name="black"/>
@@ -15,8 +18,8 @@
         <collision>
             <geometry>
-                <cylinder radius="0.05" length="0.04"/>
+                <cylinder radius="${lidar_radius}" length="${lidar_length}"/>
             </geometry>
         </collision>
-        <xacro:inertial_cylinder mass="0.1" length="0.04" radius="0.05">
+        <xacro:inertial_cylinder mass="${lidar_mass}" length="${lidar_length}" radius="${lidar_radius}">
             <origin xyz="0 0 0" rpy="0 0 0"/>
         </xacro:inertial_cylinder>
@@ -39,5 +42,5 @@
                 <range>
                     <min>0.3</min>
-                    <max>16</max>
+                    <max>12</max>
                     <resolution>0.01</resolution>
                 </range>

File: description_ackerman/ros_control.xacro (robot description, xacro)
@@ -5,5 +5,5 @@
         <plugin>gazebo_ros2_control/GazeboSystem</plugin>
       </hardware>
-      <joint name="virtual_front_wheel_joint">
+      <joint name="front_wheel_steering_joint">
         <command_interface name="position">
           <param name="min">-0.785</param>
